File: KICAD_FILES/st_link_diy/st_link_diy.kicad_sch (KiCad schematic)
At the start: 0 parts

Commit message: added schematic v0.1
Parts:
- added C? (x5): 100n, symbol Device:C
- added C? (x2): 20p, symbol Device:C
- added C?: 470p, symbol Device:C
- added C?: 1uF, symbol Device:C
- added D? (x2): LED, symbol Device:LED
- added J?: USB_B, symbol Connector:USB_B
- added J?: Conn_01x06_Male, symbol Connector:Conn_01x06_Male
- added J?: Conn_02x05_Odd_Even, symbol Connector_Generic:Conn_02x05_Odd_Even
- added JP?: Jumper_3_Bridged12, symbol Jumper:Jumper_3_Bridged12
- added Q?: BC817, Package_TO_SOT_SMD:SOT-23, symbol Transistor_BJT:BC817
- added R?: DNP, symbol Device:R
- added R?: 1M, symbol Device:R
- added R? (x2): 220, symbol Device:R
- added R? (x3): 10k, symbol Device:R
- added R? (x2): 100, symbol Device:R
- added R? (x2): 100k, symbol Device:R
- added R? (x2): 0, symbol Device:R
- added R?: 1.5k, symbol Device:R
- added R?: 36k, symbol Device:R
- added R? (x2): 4.7k, symbol Device:R
- added U?: TC1263-5.0VOATR, Microchip-TC1263-5.0VOATR-*, symbol eec:TC1263-5.0VOATR
- added U?: STM32F103CBTx, Package_QFP:LQFP-48_7x7mm_P0.5mm, symbol MCU_ST_STM32F1:STM32F103CBTx
- added Y?: 8MHz, symbol Device:Crystal
Connections:
- new net: R?.2, U?.3 (PC14)
- new net: R?.2, U?.5 (~{ERROR})
- new net: D?.2 (A), R?.2
- new net: D?.1 (K), R?.1
- new net: C?.1, U?.4 (BYPASS)
- new net: R?.2, U?.6 (~{SHDN})
- new net: J?.2 (D-), R?.1
- new net: J?.3 (D+), R?.1, R?.1
- new net: C?.2, U?.6 (PD1), Y?.1
- new net: C?.1, U?.5 (PD0), Y?.2
- new net: R?.2, U?.2 (PC13)
- new net: Q?.1 (B), R?.1, R?.1, R?.2
- new net: Q?.2 (E), R?.2
- new net: R?.2, U?.25 (PB12)
- new net: R?.1, R?.2, U?.10 (PA0)
- new net: JP?.2 (C), R?.1
- new net +3V3: C?.1, C?.1, C?.1, C?.1, C?.1, J?.1 (Pin_1), J?.2 (Pin_2), JP?.1 (A), Q?.3 (C), R?.1, R?.2, U?.1 (VBAT), U?.1 (VOUT), U?.24 (VDD), U?.36 (VDD), U?.48 (VDD), U?.9 (VDDA)
- new net +5V: J?.1 (Pin_1), J?.1 (VBUS), R?.1, R?.1, R?.2, U?.8 (VIN)
- new net BOOT0: J?.4 (Pin_4), R?.2, U?.44 (BOOT0)
- new net CLK: J?.3 (Pin_3), U?.37 (PA14)
- new net DIO: J?.2 (Pin_2), U?.34 (PA13)
- new net GND: C?.1, C?.1, C?.2, C?.2, C?.2, C?.2, C?.2, C?.2, C?.2, J?.4 (GND), J?.4 (Pin_4), J?.5 (Shield), J?.6 (Pin_6), R?.1, R?.1, R?.1, R?.1, R?.2, R?.2, U?.2 (GND), U?.23 (VSS), U?.35 (VSS), U?.47 (VSS), U?.8 (VSSA)
- new net LED: D?.1 (K), D?.2 (A), U?.30 (PA9)
- new net NRST: C?.2, J?.5 (Pin_5), R?.1, U?.7 (NRST)
- new net T_CLK: J?.5 (Pin_5), U?.26 (PB13)
- new net T_DIO: J?.6 (Pin_6), R?.1, U?.27 (PB14)
- new net T_PWR: J?.3 (Pin_3), JP?.3 (B)
- new net T_RST: J?.8 (Pin_8), U?.18 (PB0)
- new net T_RX: J?.10 (Pin_10), U?.13 (PA3)
- new net T_SWO: J?.7 (Pin_7), U?.31 (PA10)
- new net T_TX: J?.9 (Pin_9), U?.12 (PA2)
- new net USB_D+: R?.2, U?.33 (PA12)
- new net USB_D-: R?.2, U?.32 (PA11)
- new net USB_RENUM: R?.2, U?.38 (PA15)
- no-connect marks 0 -> 2
Other:
- note added: "CONN FOR PROGRAMMING"
- note added: "LED"
- note added: "STM32"
- note added: "TARGET CONN"
- note added: "USB INPUT"
- note added: "VOLTAGE REGULATOR"

Commit message: finished schematic
Parts:
- C1, C5, C6, C7, C8, C9: renamed from C?; footprint (none) -> Capacitor_SMD:C_0805_2012Metric_Pad1.18x1.45mm_HandSolder
- C2: renamed from C?; footprint (none) -> Capacitor_SMD:C_Elec_4x5.4
- C3, C4: renamed from C?; footprint (none) -> Capacitor_SMD:C_0603_1608Metric_Pad1.08x0.95mm_HandSolder
- D1, D2: renamed from D?; footprint (none) -> LED_SMD:LED_0805_2012Metric_Pad1.15x1.40mm_HandSolder
- J1: renamed from J?; footprint (none) -> Connector_USB:USB_B_OST_USB-B1HSxx_Horizontal
- J2: renamed from J?; footprint (none) -> Connector_IDC:IDC-Header_2x05_P2.54mm_Vertical
- J3: renamed from J?; footprint (none) -> Connector_PinHeader_2.54mm:PinHeader_1x06_P2.54mm_Vertical
- JP1: renamed from JP?; footprint (none) -> Connector_PinHeader_2.54mm:PinHeader_1x03_P2.54mm_Vertical
- R1, R10, R11, R12, R13, R14, R15, R16, R17, R2, R3, R4, R5, R6, R7, R8, R9: renamed from R?; footprint (none) -> Resistor_SMD:R_1206_3216Metric_Pad1.30x1.75mm_HandSolder
- U1: renamed from U?; footprint Microchip-TC1263-5.0VOATR-* -> Package_SO:SOIC-8-1EP_3.9x4.9mm_P1.27mm_EP2.29x3mm
- Y1: renamed from Y?; footprint (none) -> Crystal:Crystal_SMD_HC49-SD_HandSoldering
- gave numbers to parts that had none: 2
Connections:
- no-connect marks 2 -> 21
