File: KICAD_FILES/st_link_diy/st_link_diy.kicad_pcb (KiCad board)
At the start: 2 copper layers, 36 parts, among them J1 USB_B, J2 Conn_02x05_Odd_Even, J3 Conn_01x06_Male, Q1 BC817, U1 TC1263-5.0VOATR, U2 STM32F103CBTx, Y1 8MHz

Commit message: added pcb
Parts:
- moved U1 90.0 mm to (96.5, 172.7)
- moved C2 80.6 mm to (104.5, 172.4)
- moved R4 69.0 mm to (162.6, 106.7)
- moved C4 65.5 mm to (166.0, 154.3)
- moved R3 62.4 mm to (153.3, 89.3)
- moved R2 58.3 mm to (154.9, 151.7)
- moved J2 58.2 mm to (152.4, 116.8)
- moved R17 53.7 mm to (160.9, 151.7)
- moved R12 51.6 mm to (154.9, 154.9)
- moved R11 50.4 mm to (160.9, 154.9)
- moved C9 50.2 mm to (166.3, 151.5)
- moved R8 46.1 mm to (165.2, 89.3)
- moved J1 42.5 mm to (72.6, 120.6), turned to 180 degrees
- moved R7 37.5 mm to (159.3, 89.3)
- moved Y1 34.6 mm to (105.0, 154.9)
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